File: Hardware/Motherboard/KiCad/Motherboard.kicad_pcb (KiCad board)
At the start: 2 copper layers, 0 parts

Commit message: Motherboard PCB Rev. 1.0
Parts:
- added BZ1: Buzzer, Connector_PinHeader_2.54mm:PinHeader_1x02_P2.54mm_Vertical, B.Cu at (133.0, 128.0)
- added C1: 10nF, Capacitor_SMD:C_1206_3216Metric_Pad1.33x1.80mm_HandSolder, F.Cu at (138.5, 126.4)
- added C2: 100uF, Capacitor_SMD:CP_Elec_6.3x5.4, F.Cu at (159.5, 128.7)
- added D1: 1N4148WS, Diode_SMD:D_SOD-323_HandSoldering, F.Cu at (131.8, 125.0)
- added H1: M3, MountingHole:MountingHole_3.2mm_M3_Pad_Via, F.Cu at (106.6, 129.4)
- added H2: M3, MountingHole:MountingHole_3.2mm_M3_Pad_Via, F.Cu at (189.9, 129.4)
- added J1: USB, Footprints:USB_Pin_Header, B.Cu at (148.2, 131.5)
- added J2: FOLLOWER TUBE(S), Connector_PinHeader_2.54mm:PinHeader_1x03_P2.54mm_Vertical, B.Cu at (182.5, 131.5)
- added J3: MAIN TUBE(S), Connector_PinHeader_2.54mm:PinHeader_1x03_P2.54mm_Vertical, B.Cu at (172.0, 131.5)
- added Q1: MMBT3904, Package_TO_SOT_SMD:SOT-23_Handsoldering, F.Cu at (126.0, 128.0)
- added Q2: MMBT3904, Package_TO_SOT_SMD:SOT-23_Handsoldering, F.Cu at (178.9, 114.5)
- added Q3: MMBT3904, Package_TO_SOT_SMD:SOT-23_Handsoldering, F.Cu at (170.9, 114.5)
- added Q4: MMBT3904, Package_TO_SOT_SMD:SOT-23_Handsoldering, F.Cu at (174.9, 107.5)
- added Q5: MMBT3904, Package_TO_SOT_SMD:SOT-23_Handsoldering, F.Cu at (178.9, 107.5)
- added Q6: MMBT3904, Package_TO_SOT_SMD:SOT-23_Handsoldering, F.Cu at (182.9, 107.5)
- added Q7: MMBT3906, Package_TO_SOT_SMD:SOT-23_Handsoldering, F.Cu at (182.9, 114.5)
- added Q8: MMBT3906, Package_TO_SOT_SMD:SOT-23_Handsoldering, F.Cu at (174.9, 114.5)
- added R1: (Current Limit / Volume Adj.), Resistor_SMD:R_1206_3216Metric_Pad1.30x1.75mm_HandSolder, F.Cu at (136.0, 126.5)
- added R10: 10k, Resistor_SMD:R_1206_3216Metric_Pad1.30x1.75mm_HandSolder, F.Cu at (175.0, 121.5)
- added R11: 10k, Resistor_SMD:R_1206_3216Metric_Pad1.30x1.75mm_HandSolder, F.Cu at (178.0, 102.0)
- added R12: 10k, Resistor_SMD:R_1206_3216Metric_Pad1.30x1.75mm_HandSolder, F.Cu at (175.5, 102.0)
- added R13: 10k, Resistor_SMD:R_1206_3216Metric_Pad1.30x1.75mm_HandSolder, F.Cu at (180.5, 102.0)
- added R14: 10k, Resistor_SMD:R_1206_3216Metric_Pad1.30x1.75mm_HandSolder, F.Cu at (183.0, 102.0)
- added R2: 1k, Resistor_SMD:R_1206_3216Metric_Pad1.30x1.75mm_HandSolder, F.Cu at (122.0, 126.5)
- added R3: 10k, Resistor_SMD:R_1206_3216Metric_Pad1.30x1.75mm_HandSolder, F.Cu at (182.1, 127.0)
- added R4: 10k, Resistor_SMD:R_1206_3216Metric_Pad1.30x1.75mm_HandSolder, F.Cu at (171.6, 127.0)
- added R5: 10k, Resistor_SMD:R_1206_3216Metric_Pad1.30x1.75mm_HandSolder, F.Cu at (179.0, 121.5)
- added R6: 10k, Resistor_SMD:R_1206_3216Metric_Pad1.30x1.75mm_HandSolder, F.Cu at (181.5, 121.5)
- added R7: 10k, Resistor_SMD:R_1206_3216Metric_Pad1.30x1.75mm_HandSolder, F.Cu at (170.0, 121.5)
- added R8: 10k, Resistor_SMD:R_1206_3216Metric_Pad1.30x1.75mm_HandSolder, F.Cu at (172.5, 121.5)
- added R9: 10k, Resistor_SMD:R_1206_3216Metric_Pad1.30x1.75mm_HandSolder, F.Cu at (184.0, 121.5)
- added U1: ~, Footprints:YD-ESP32-S3_(ESP32-S3-DevKitC-1_USB-C_Clone), F.Cu at (161.1, 93.6)
- added U2: ~, Footprints:3.2in_SPI_TFT_Touch_Screen_&_SD_Card_Module, F.Cu at (103.1, 37.1)
Routing:
- net +5V: track 0.00 -> 269.7 mm
- net SCLK: track 0.00 -> 148.2 mm
- net MISO: track 0.00 -> 133.9 mm
- net MOSI: track 0.00 -> 120.6 mm
- net +3V3: track 0.00 -> 96.1 mm, vias 0 -> 12
- net FOLLOWER_TRG: track 0.00 -> 86.9 mm
- net SD_CD: track 0.00 -> 76.2 mm
- net COINCIDENCE_TRG: track 0.00 -> 72.8 mm
- net MAIN_TRG: track 0.00 -> 61.8 mm
- net DISPLAY_CS: track 0.00 -> 53.2 mm
- net DISPLAY_RST: track 0.00 -> 49.6 mm
- net Net-(J1-Pin_3): track 0.00 -> 48.2 mm
- net DISPLAY_DC: track 0.00 -> 46.0 mm
- net Net-(J1-Pin_2): track 0.00 -> 44.4 mm
- net DISPLAY_LED: track 0.00 -> 39.1 mm
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- added copper zone on B.Cu, net GND
- added copper zone on F.Cu, net GND
Other:
- board outline added: 94.5 x 100 mm
- board text added: "+"
- board text added: "+5V"
- board text added: "3.2in SPI TFT Touch Screen & SD Card Module Resolution: 240x320 px Display driver: ILI9341 Touch driver: XPT2046"
- board text added: ": Motherboard : 1.0 : 2024-09-08"
- board text added: "BUZZER"
- board text added: "DATA+"
- board text added: "DATA-"
- board text added: "FOLLOWER T."
- board text added: "GMT Geiger Counter Motherboard Rev. 1.0 Median Dispersion 2024 https://github.com/median-dispersion/GMT-Geiger-Counter"
- board text added: "GND"
- board text added: "MAIN TUBE(S)"
- board text added: "PCB REV DAT"
- board text added: "PULSE"
- board text added: "USB"
- board text added: "YD-ESP32-S3"

Commit message: Added BoM for motherboard
Parts:
- U1: value ~ -> YD-ESP32-S3 N16R8 (ESP32-S3-DevKitC-1 USB-C Clone)
- U2: value ~ -> MSP3218
Other:
- board text added: ": Motherboard : 1.0 : 2024-09-10"
- board text removed: ": Motherboard : 1.0 : 2024-09-08"

Commit message: Fixed disconnected pad
Routing:
- net MOSI: track 120.6 -> 165.7 mm
- net DISPLAY_DC: track 46.0 -> 47.6 mm
- net DISPLAY_RST: track 49.6 -> 51.1 mm
- net DISPLAY_CS: track 53.2 -> 54.7 mm
- net GND: vias 58 -> 57
Changed lines of the file:
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@@
-	)
-	(via
-		(at 124.5 93.5)
-		(size 0.5)
-		(drill 0.3)
-		(layers "F.Cu" "B.Cu")
-		(free yes)
-		(net 4)
 	)
 	(via
@@
 	(segment
 		(start 105.6 58.75)
-		(end 128.29 81.44)
+		(end 108.25 58.75)
 		(width 0.3)
 		(layer "F.Cu")
@@
 	)
 	(segment
-		(start 128.29 81.44)
+		(start 108.25 58.75)
+		(end 128.29 78.79)
+		(width 0.3)
+		(layer "F.Cu")
+		(net 27)
+	)
+	(segment
+		(start 128.29 78.79)
 		(end 128.29 95.35)
 		(width 0.3)
@@
 	)
 	(segment
+		(start 124.5 97)
+		(end 118.5 97)
+		(width 0.3)
+		(layer "F.Cu")
+		(net 30)
+	)
+	(segment
 		(start 137.173338 82.826662)
 		(end 137.173338 96.326662)
@@
 	)
 	(segment
+		(start 124.5 77.5)
+		(end 124.5 97)
+		(width 0.3)
+		(layer "F.Cu")
+		(net 30)
+	)
+	(segment
 		(start 108.53 76.53)
 		(end 118.13 86.13)
@@
 	)
 	(segment
-		(start 136.5 97)
-		(end 118.5 97)
-		(width 0.3)
-		(layer "F.Cu")
-		(net 30)
-	)
-	(segment
 		(start 189.9 63.83)
 		(end 156.17 63.83)
@@
 	)
 	(segment
+		(start 136.5 97)
+		(end 124.5 97)
+		(width 0.3)
+		(layer "F.Cu")
+		(net 30)
+	)
+	(segment
 		(start 118.13 96.63)
 		(end 118.13 95.35)
@@
 	)
 	(segment
-		(start 133.37 81.44)
+		(start 108.29 61.29)
+		(end 124.5 77.5)
+		(width 0.3)
+		(layer "F.Cu")
+		(net 30)
+	)
+	(segment
+		(start 105.6 61.29)
+		(end 108.29 61.29)
+		(width 0.3)
+		(layer "F.Cu")
+		(net 30)
+	)
+	(segment
+		(start 105.6 53.67)
+		(end 108.17 53.67)
+		(width 0.3)
+		(layer "F.Cu")
+		(net 34)
+	)
+	(segment
+		(start 133.37 78.87)
 		(end 133.37 95.35)
 		(width 0.3)
@@
 	)
 	(segment
-		(start 105.6 53.67)
-		(end 133.37 81.44)
+		(start 108.17 53.67)
+		(end 133.37 78.87)
 		(width 0.3)
 		(layer "F.Cu")
@@
 	)
 	(segment
-		(start 130.83 81.44)
+		(start 105.6 56.21)
+		(end 108.21 56.21)
+		(width 0.3)
+		(layer "F.Cu")
+		(net 46)
+	)
+	(segment
+		(start 108.21 56.21)
+		(end 130.83 78.83)
+		(width 0.3)
+		(layer "F.Cu")
+		(net 46)
+	)
+	(segment
+		(start 130.83 78.83)
 		(end 130.83 95.35)
 		(width 0.3)
 		(layer "F.Cu")
-		(net 46)
-	)
-	(segment
-		(start 105.6 56.21)
-		(end 130.83 81.44)
-		(width 0.3)
-		(layer "F.Cu")
