File: Hardware/Motherboard/KiCad/Motherboard.kicad_pcb (KiCad board)
At the start: 2 copper layers, 94.5 x 100 mm, 33 parts, among them J1 USB, J2 FOLLOWER TUBE(S), J3 MAIN TUBE(S), Q1 MMBT3904, Q2 MMBT3904, Q3 MMBT3904, Q4 MMBT3904, Q5 MMBT3904, Q6 MMBT3904, Q7 MMBT3906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

Commit message: Changed component value, fixed typos & fixed small mistakes
Connections:
- net SD_CD renamed SD_CS
Changed lines of the file:
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@@
 	(title_block
 		(title "Motherboard")
-		(date "2024-09-10")
+		(date "2024-11-14")
 		(rev "1.0")
 		(company "https://github.com/median-dispersion/GMT-Geiger-Counter")
@@
 	(net 24 "unconnected-(U1-TX-Pad43)")
 	(net 25 "unconnected-(U1-Pad5)")
-	(net 26 "SD_CD")
+	(net 26 "SD_CS")
 	(net 27 "DISPLAY_DC")
 	(net 28 "unconnected-(U1-48-Pad29)")
@@
 			(layers "*.Cu" "*.Mask")
 			(remove_unused_layers no)
-			(net 26 "SD_CD")
+			(net 26 "SD_CS")
 			(pinfunction "17")
 			(pintype "input")
@@
 			(layers "*.Cu" "*.Mask")
 			(remove_unused_layers no)
-			(net 26 "SD_CD")
+			(net 26 "SD_CS")
 			(pinfunction "SD_CS")
 			(pintype "input")
