File: Hardware/Tube Driver/KiCad/Tube Driver.kicad_pcb (KiCad board)
At the start: 2 copper layers, 157.5 x 30.5 mm, 45 parts, among them J1 I/O, Q1 MMBT3904, Q2 STN2580, Q3 MMBT3904, Q4 MMBT3906, U1 NE555D

Commit message: Fixed component value typo
Parts:
- C5, C6: value 47pF -> 47nF
Other:
- board text added: ": Tube Driver : 1.0 : 2024-09-10"
- board text removed: ": Tube Driver : 1.0 : 2024-09-06"
Changed lines of the file:
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@@
 	(title_block
 		(title "Tube Driver")
-		(date "2024-09-06")
+		(date "2024-09-10")
 		(rev "1.0")
 		(company "https://github.com/median-dispersion/GMT-Geiger-Counter")
@@
 			)
 		)
-		(property "Value" "47pF"
+		(property "Value" "47nF"
 			(at 0 2.5 -90)
 			(layer "F.Fab")
@@
 			)
 		)
-		(property "Value" "47pF"
+		(property "Value" "47nF"
 			(at 0 -3 -90)
 			(layer "F.Fab")
@@
 		)
 	)
-	(gr_text ": Tube Driver\n: 1.0\n: 2024-09-06"
+	(gr_text ": Tube Driver\n: 1.0\n: 2024-09-10"
 		(at 215.8 104 90)
 		(layer "B.SilkS")
